File: KiCad Projeto Tractian/fullWirelessComTractian.kicad_sch (KiCad schematic)
At the start: 28 parts, among them U1 ESP8266EX, U2 AT25SF081-SSHD-X, U4 MX25R3235FM2xx1, U5 AMS1117-3.3, U6 TMP36xS, Y2 XTAL 16Mhz ±10ppm (TSX -3225 )

Commit message: :rocket: Rotina de leitura de temperatura com estabilizacao por filtro LTI media movel
Changed lines of the file:
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@@
   )
   (symbol (lib_id "Memory_Flash:AT25SF081-SSHD-X") (at 251.46 52.07 0) (unit 1)
-    (in_bom yes) (on_board yes) (dnp no) (fields_autoplaced)
-    (property "Reference" "U2" (at 260.35 51.435 0)
+    (in_bom yes) (on_board yes) (dnp no)
+    (property "Reference" "U2" (at 255.27 40.64 0)
       (effects (font (size 1.27 1.27)) (justify left))
     )
-    (property "Value" "AT25SF081-SSHD-X" (at 260.35 53.975 0)
+    (property "Value" "AT25SF081-SSHD-X" (at 260.35 62.23 90)
       (effects (font (size 1.27 1.27)) (justify left))
     )

Commit message: :rocket: Read (right this time) 1024 bytes of data Function
Parts:
- U6: value TMP36xS -> TMP35
Changed lines of the file:
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@@
       (effects (font (size 1.27 1.27)))
     )
-    (property "Value" "TMP36xS" (at 236.22 139.7 0)
+    (property "Value" "TMP35" (at 236.22 139.7 0)
       (effects (font (size 1.27 1.27)))
     )

Commit message: :memo: Updates on the documentation | Preliminares, Introduction and Part of Schematics and PCB Design
Other:
- note added: "Storage Circuitry"
- note removed: "Program & Data Memory"
Changed lines of the file:
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@@
     (effects (font (size 5 5)) (justify left bottom))
   )
-  (text "Program & Data Memory\n\n" (at 189.23 29.21 0)
+  (text "Storage Circuitry\n" (at 189.23 21.59 0)
     (effects (font (size 5 5)) (justify left bottom))
   )
